File: pcb/a4988_driver.kicad_sch (KiCad schematic)
At the start: 3 parts, among them U2 A4988SETTR-T

Commit message: worked on a4988
Parts:
- removed R5: R, symbol Device:R
- added C2: C, symbol Device:C
- added C3, C5: 0.1uf, symbol Device:C
- added C4: 100uf, symbol Device:C
- added C_small, C_small_2: 0.1uf, symbol Device:C_Small
- added R6: 20k, symbol Device:R
- added R7: Potentiometer, symbol Simulation_SPICE:Potentiometer
- added R8, R9: 0.05, symbol Device:R
- C1: value 0.1μ -> 0.22uf
Connections:
- net GND: now also C1.2, U2.18 (GND), U2.29, C2.1, C4.2, R6.1, R7.3, R8.2, R9.2
- net at U2.5 (CP2): now also C_small_2.2; no longer C1.1
- net at U2.4 (CP1): now also C_small_2.1; no longer C1.2
- net +5V: now reaches U2.12 (*RESET)
- net +5V: now also C1.1, U2.14 (*SLEEP), C5.2, R7.1
- net at U2.13 (ROSC): now also R6.2
- net at U2.15 (VDD): now also C5.1
- net at U2.17 (REF): now also R7.2
- net at U2.22 (VBB1): now also U2.28 (VBB2), C3.2, C4.1
- net at U2.23 (SENSE1): now also R8.1
- net at U2.27 (SENSE2): now also R9.1
- net at U2.6 (VCP): now also C_small.1
- net at U2.8 (VREG): now also C2.2
- new net +12V: C3.1, C_small.2

Commit message: added shift register bom and a4988
Parts:
- added C6: C, symbol Device:C
- added J2: Conn_01x04_Pin, symbol Connector:Conn_01x04_Pin
- added J3: Barrel_Jack, symbol Connector:Barrel_Jack
- renumbered C_small to C_small1
Connections:
- net +12V: now also C6.1, J3.1
- net GND: now also C6.2, J3.2
- net OUT2B A4988: now reaches U2.1 (OUT2B)
- net OUT2B A4988: now also J2.1 (Pin_1)
- net MS2 A4988: now reaches U2.10 (MS2)
- net MS3 A4988: now reaches U2.11 (MS3)
- net STEP A4988: now reaches U2.16 (STEP)
- net DIR A4988: now reaches U2.19 (DIR)
- net OUT1B A4988: now reaches U2.21 (OUT1B)
- net OUT1B A4988: now also J2.4 (Pin_4)
- net OUT1A A4988: now reaches U2.24 (OUT1A)
- net OUT1A A4988: now also J2.3 (Pin_3)
- net OUT2A A4988: now reaches U2.26 (OUT2A)
- net OUT2A A4988: now also J2.2 (Pin_2)
- net MS1 A4988: now reaches U2.9 (MS1)
Other:
- moved on the sheet: C1, C2, C3, C4, C5, C_small1, C_small_2, R6, R7, R8, R9, U2

Commit message: added journal, and more pcb stuff
Connections:
- net +12V: now also U2.22 (VBB1), U2.28 (VBB2)
- net +5V: now also C5.1, U2.15 (VDD); no longer C1.1, C5.2
- net GND: now also U2.2 (*ENABLE), U2.3 (GND)
- net at C3.2, C4.1: no longer U2.22 (VBB1), U2.28 (VBB2)
- new net: C1.1, C5.2
Other:
- moved on the sheet: C1, C3
